Commit message: 最新版

File: sobit_model/urdf/sobit.urdf (robot description, URDF)
Before this commit: robot sobit, 14 links, 13 joints
Links:
- added link left_hand; visual mesh filename=package://sobit_model/mesh/SOBIT_hand.stl
- added link left_hand_index; visual mesh filename=package://sobit_model/mesh/SOBIT_index.stl
- added link left_hand_middle; visual mesh filename=package://sobit_model/mesh/SOBIT_index.stl scale=1 1 1.0588
- added link left_hand_pinky; visual mesh filename=package://sobit_model/mesh/SOBIT_index.stl scale=1 1 0.88
- added link left_hand_ring; visual mesh filename=package://sobit_model/mesh/SOBIT_index.stl scale=1 1 1
- added link left_hand_thumb; visual mesh filename=package://sobit_model/mesh/SOBIT_thumb.stl
- added link right_hand; visual mesh filename=package://sobit_model/mesh/SOBIT_hand_right.stl
- added link right_hand_thumb; visual mesh filename=package://sobit_model/mesh/SOBIT_thumb_right.stl
- added link right_hand_twist; visual box size=0.06 0.01 0.07
- link left_wheel: geometry visual mesh filename=package://sobit_model/mesh/wheel.stl
Joints:
- added joint left_hand_index: type revolute, parent left_hand, child left_hand_index, origin xyz=0.04 -0.01 -0.09 rpy=0 0 0, axis 1 0 0, limit lower=-1.571 upper=0 effort=1000 velocity=0.5
- added joint left_hand_middle: type revolute, parent left_hand, child left_hand_middle, origin xyz=0.02 -0.01 -0.09 rpy=0 0 0, axis 1 0 0, limit lower=-1.571 upper=0 effort=1000 velocity=0.5
- added joint left_hand_pinky: type revolute, parent left_hand, child left_hand_pinky, origin xyz=-0.02 -0.01 -0.09 rpy=0 0 0, axis 1 0 0, limit lower=-1.571 upper=0 effort=1000 velocity=0.5
- added joint left_hand_ring: type revolute, parent left_hand, child left_hand_ring, origin xyz=0 -0.01 -0.09 rpy=0 0 0, axis 1 0 0, limit lower=-1.571 upper=0 effort=1000 velocity=0.5
- added joint left_hand_thumb: type revolute, parent left_hand, child left_hand_thumb, origin xyz=0.04 -0.035 -0.055 rpy=0 0 0, axis 0 -1 0, limit lower=-1.571 upper=1.571 effort=1000 velocity=0.5
- added joint left_hand_wrist: type revolute, parent left_second_arm, child left_hand, origin xyz=0 0.04 -0.17 rpy=0 0 1.571, axis 0 0 1, limit lower=-1.571 upper=1.571 effort=1000 velocity=0.5
- added joint right_arm_to_right_hand: type fixed, parent right_second_arm, child right_hand, origin xyz=0 -0.04 -0.17 rpy=0 0 1.571
- added joint right_hand_to_right_thumb: type fixed, parent right_hand, child right_hand_thumb, origin xyz=-0.04 -0.035 -0.055 rpy=0 0 0
- added joint right_hand_twist: type revolute, parent right_hand, child right_hand_twist, origin xyz=-0.02 -0.01 -0.09 rpy=0 0 0, axis 1 0 0, limit lower=-1.571 upper=0 effort=1000 velocity=0.5
- joint left_elbow_yaw: origin xyz=0.00 0 -0.175 rpy=0 0 0 -> xyz=0.00 0 -0.175 rpy=0 0 -1.571
- joint left_shoulder_roll: origin xyz=0.00 0.075 0 rpy=0.1 0 0 -> xyz=0.00 0.075 0 rpy=0.0 0 0
- joint right_elbow_yaw: origin xyz=0.00 0 -0.175 rpy=0 0 0 -> xyz=0.00 0 -0.175 rpy=0 0 1.571
- joint right_shoulder_roll: origin xyz=0.00 -0.075 0 rpy=-0.1 0 0 -> xyz=0.00 -0.075 0 rpy=0.0 0 0
